File: TampanMD.kicad_pcb (KiCad board)
At the start: 2 copper layers, 50 x 50 mm, 93 parts, among them J1 Conn_01x10, U1 F2800132RHBR, U10 BSC009NE2LS, U11 AMC1301DWVR, U12 TLV62130, U2 UCC27211DRMR, U3 UCC27211DRMR, U4 UCC27211DRMR, U5 BSC009NE2LS, U6 BSC009NE2LS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

Commit message: Update TampanMD.kicad_pcb
Routing:
- net ISENSE_N: track 143.9 -> 161.1 mm, vias 41 -> 40
- net VDD: track 141.7 -> 156.5 mm
- net EPWM2_B: track 17.6 -> 19.0 mm
- net Net-(U4-LO): track 9.53 -> 8.44 mm
- net Net-(R5-Pad1): track 20.2 -> 20.7 mm
- net MCU_A_3V3: track 29.1 -> 29.6 mm, vias 6 -> 5
- added copper zone on B.Cu, net VDD
Other:
- board text added: "Aziz Faozi"

Commit message: Update TampanMD.kicad_pcb
Parts:
- moved C6 0.08 mm to (128.0, 92.0)
Routing:
- net VDD: track 156.5 -> 174.6 mm, vias 35 -> 38

Commit message: Update TampanMD.kicad_pcb
Routing:
- net ISENSE_N: track 161.3 -> 162.4 mm
Changed lines of the file:
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@@
 		(tags "capacitor")
 		(property "Reference" "C9"
-			(at 1.77 0.87 0)
+			(at 1.81 -0.09 0)
 			(layer "F.SilkS")
 			(effects
@@
 	)
 	(segment
+		(start 124.59 89.5)
+		(end 124.64 89.55)
+		(width 0.2)
+		(layer "F.Cu")
+		(net 48)
+	)
+	(segment
 		(start 117.55 70.3)
 		(end 117.95 70.3)
@@
 	)
 	(segment
+		(start 123.5 89.5)
+		(end 124.59 89.5)
+		(width 0.2)
+		(layer "F.Cu")
+		(net 48)
+	)
+	(segment
 		(start 126.963282 67.95)
 		(end 128.1 67.95)
@@
 	)
 	(segment
-		(start 124.64 89.55)
-		(end 124.03 88.94)
-		(width 0.2)
-		(layer "F.Cu")
-		(net 48)
-	)
-	(segment
 		(start 112.45 59.3)
 		(end 112.45 59.85)
@@
 	)
 	(segment
-		(start 124.64 89.86)
-		(end 124.64 89.55)
-		(width 0.2)
-		(layer "F.Cu")
-		(net 48)
-	)
-	(segment
 		(start 117.1 87.3)
 		(end 115.649943 87.3)
@@
 	)
 	(segment
+		(start 124.64 89.55)
+		(end 124.64 89.86)
+		(width 0.2)
+		(layer "F.Cu")
+		(net 48)
+	)
+	(segment
 		(start 122.175 91.875)
 		(end 122.5 92.2)
@@
 	)
 	(via
-		(at 124.03 88.94)
+		(at 123.5 89.5)
 		(size 0.6)
 		(drill 0.3)
@@
 	)
 	(segment
-		(start 124.03 88.94)
-		(end 124.03 88.42)
-		(width 0.2)
-		(layer "B.Cu")
-		(net 48)
-	)
-	(segment
 		(start 137.969265 91.359265)
 		(end 135.475999 88.865999)
@@
 	)
 	(segment
-		(start 124.03 88.42)
-		(end 124.15 88.3)
+		(start 117.93389 62.98389)
+		(end 117.93389 65.125507)
 		(width 0.2)
 		(layer "B.Cu")
@@
 	)
 	(segment
-		(start 117.93389 62.98389)
-		(end 117.93389 65.125507)
+		(start 124.03 88.97)
+		(end 124.03 88.42)
 		(width 0.2)
 		(layer "B.Cu")
@@
 		(width 0.2)
 		(layer "B.Cu")
+		(net 48)
+	)
+	(segment
+		(start 123.5 89.5)
+		(end 124.03 88.97)
+		(width 0.2)
+		(layer "B.Cu")
+		(net 48)
+	)
+	(segment
+		(start 124.03 88.42)
+		(end 124.15 88.3)
+		(width 0.2)
+		(layer "B.Cu")

Commit message: done i guess
Parts:
- added R34: 10K, Resistor_SMD:R_0603_1608Metric, F.Cu at (116.9, 79.3)
- added R35: 10K, Resistor_SMD:R_0603_1608Metric, F.Cu at (116.8, 83.2)
- moved R33 0.21 mm to (116.4, 81.7)
Routing:
- net /MCU/I2CB_SCL: track 18.3 -> 24.0 mm
- net 3V3: track 99.1 -> 103.6 mm
- net /MCU/I2CB_SDA: track 18.8 -> 19.6 mm
- net Net-(U1-GPIO32): track 19.5 -> 20.1 mm
- net /MCU/CANA_TX: track 28.8 -> 29.4 mm
