File: mcu.kicad_sch (KiCad schematic)
At the start: 30 parts, among them J1 Conn_01x10, U1 F2800132RHBR, U11 AMC1301DWVR, Y1 X322520MSB4SI

Commit message: done i guess
Parts:
- added R34, R35: 10K, Resistor_SMD:R_0603_1608Metric, symbol Device:R_US
Connections:
- net 3V3: now also R34.1, R35.1
- net I2CB_SCL: now also R35.2
- net I2CB_SDA: now also R34.2
